Commit message: Fix some syntax deprecation warnings

File: lwr_description/model/kuka_lwr.transmission.xacro (robot description, xacro)
@@ -1,6 +1,6 @@
 <?xml version="1.0"?>
 <robot xmlns:xacro="http://www.ros.org/wiki/xacro">
-	<xacro:property name="Interface10" value="PositionJointInterface"/>
-	<xacro:property name="Interface30" value="EffortJointInterface"/>
+  <xacro:property name="Interface10" value="hardware_interface/PositionJointInterface"/>
+  <xacro:property name="Interface30" value="hardware_interface/EffortJointInterface"/>
 	<xacro:macro name="kuka_lwr_transmission" params="name">
 		<transmission name="${name}_a1_trans">
